File: hardware/picoPD_interrogator/typec_1.kicad_sch (KiCad schematic)
At the start: 31 parts, among them J2 USB_C_Receptacle_USB2.0_16P, Q1 rohm-RE1C002UN, Q2 rohm-RE1C002UN, Q4 rohm-RE1C002UN, Q5 rohm-RE1C002UN, U3 ST-LM393QT, U4 TI_SN74LVC1G3157-Q1, U5 TI_SN74LVC1G3157-Q1

Commit message: Working on schematic.
Other:
- note added: "Interrogation Port 1 [USB-C receptacle]"
- note added: "Port 1 is configured with Rd resistors. (Default Role: UFP)"
- note removed: "Interrogation Port 2 [USB-C receptacle]"
- note removed: "Port 2 is configured with Rd resistors. (Default Role: UFP)"
Changed lines of the file:
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@@
 		)
 	)
-	(text "Port 2 is configured with Rd resistors.\n(Default Role: UFP)"
+	(text "Port 1 is configured with Rd resistors.\n(Default Role: UFP)"
 		(exclude_from_sim no)
 		(at 48.26 184.658 0)
@@
 		)
 	)
-	(text "Interrogation Port 2\n[USB-C receptacle]"
+	(text "Interrogation Port 1\n[USB-C receptacle]"
 		(exclude_from_sim no)
 		(at 135.128 22.86 0)
