File: hardware/picoPD_interrogator/leds.kicad_sch (KiCad schematic)
At the start: 12 parts

Commit message: Updated schematic/BOM.
Parts:
- D10, D11, D12, D13, D14, D3, D4, D5, D6, D7, D8, D9: footprint LED_SMD:LED_WS2812B_PLCC4_5.0x5.0mm_P3.2mm -> picoPD_interrogator:LED_WS2812B_1.3x1.3mm; DigiKey PN (none) -> 160-LTST-E133HEGBKCT-ND; Manufacturer (none) -> Lite-On Inc.; Manufacturer PN (none) -> LTST-E133HEGBK
